Commit message: Articulate Cart v1.1

File: robots/cart/cart.urdf (robot description, URDF)
Before this commit: robot Cart, 18 links, 17 joints
Links:
- link chassis_middle: geometry collision box size=.44 .43 .02; visual box size=.44 .43 .02
- link chassis_top: geometry collision box size=.44 .43 .02; visual box size=.44 .43 .02
Joints:
- joint lb_leg_chassis_top: origin xyz=-0.215 0.22 0 rpy=0 0 0 -> xyz=-0.22 0.215 0 rpy=0 0 0
- joint left_handler_chassis_top: origin xyz=-0.215 0.22 0 rpy=0 -1.18 0 -> xyz=-0.22 0.215 0 rpy=0 -1.18 0
- joint lf_leg_chassis_top: origin xyz=0.215 0.22 0 rpy=0 0 0 -> xyz=0.22 0.215 0 rpy=0 0 0
- joint rb_leg_chassis_top: origin xyz=-0.215 -0.22 0 rpy=0 0 0 -> xyz=-0.22 -0.215 0 rpy=0 0 0
- joint rf_leg_chassis_top: origin xyz=0.215 -0.22 0 rpy=0 0 0 -> xyz=0.22 -0.215 0 rpy=0 0 0
- joint right_handler_chassis_top: origin xyz=-0.215 -0.22 0 rpy=0 -1.18 0 -> xyz=-0.22 -0.215 0 rpy=0 -1.18 0

Commit message: Finish creating fake arm server and cart joints server

File: robots/cart/cart.urdf (robot description, URDF)
Before this commit: robot Cart, 18 links, 17 joints
Links:
- removed link base_link
- added link cart_base_link
- link left_back_caster: mass None -> 0.1
- link left_back_wheel: mass None -> 0.1
- link left_front_caster: mass None -> 0.1
- link left_front_wheel: mass None -> 0.1
- link right_back_caster: mass None -> 0.1
- link right_back_wheel: mass None -> 0.1
- link right_front_caster: mass None -> 0.1
- link right_front_wheel: mass None -> 0.1
Joints:
- joint chassis_middle_base_link: parent base_link -> cart_base_link
- joint chassis_top_base_link: parent base_link -> cart_base_link
